Commit message: edited so its works

File: robotiq_description/urdf/robotiq_2f_140_config.urdf.xacro (robot description, xacro)
@@ -2,17 +2,17 @@
 <!-- Standalone URDF xacro that instantiates crab_claw_v1 -->
 <robot xmlns:xacro="http://www.ros.org/wiki/xacro" name="robotiq_2f_140">
-    <xacro:include filename="$(find bam_descriptions)/urdf/common.xacro" />
-    <xacro:arg name="config_file_path" default="$(find robotiq_description)/urdf/config/robotiq_2f_140_2f_140_v0.0.0.yaml"/>
-    <xacro:property name="config_file_path" value="$(arg config_file_path)"/>
-    <xacro:property name="cfg" value="${xacro.load_yaml(config_file_path)}"/>
+    <xacro:arg name="robotiq_description" default="$(env ROBOTIQ_DESCRIPTION_PATH)"/>
+    <xacro:arg name="config_file" default="$(arg robotiq_description)/urdf/config/robotiq_2f_140_2f_140_v0.0.0.yaml"/>
+    <xacro:property name="config_file" value="$(arg config_file)"/>
+    <xacro:property name="cfg" value="${xacro.load_yaml(config_file)}"/>
     <xacro:property name="plugin" value="${cfg['plugin']}" />
-    <xacro:property name="reflect" value="${cfg['reflect']}" />
-    <xacro:property name="prefix" value="${cfg['prefix']}" />
-    <xacro:property name="world_xyz" value="${cfg['world_xyz']}" />
-    <xacro:property name="world_rpy" value="${cfg['world_rpy']}" />
-    <xacro:property name="base_xyz" value="${cfg['base_xyz']}" />
-    <xacro:property name="base_rpy" value="${cfg['base_rpy']}" />
+    <xacro:property name="reflect" value="${cfg['args']['reflect']}" />
+    <xacro:property name="prefix" value="${cfg['info']['prefix']}" />
+    <xacro:property name="world_xyz" value="${cfg['args']['world_xyz']}" />
+    <xacro:property name="world_rpy" value="${cfg['args']['world_rpy']}" />
+    <xacro:property name="base_xyz" value="${cfg['args']['base_xyz']}" />
+    <xacro:property name="base_rpy" value="${cfg['args']['base_rpy']}" />
     <xacro:if value="${plugin != 'none'}">
-        <xacro:include filename="$(find robotiq_description)/urdf/robotiq_2f_140.ros2_control.xacro"/>
+        <xacro:include filename="$(arg robotiq_description)/urdf/robotiq_2f_140.ros2_control.xacro"/>
         <xacro:gripper_v1_ros2_control prefix="${prefix}" plugin="${plugin}"/>
     </xacro:if>
@@ -29,5 +29,5 @@
         <child link="${prefix}robotiq_140_base_link"/>
     </joint>
-    <xacro:include filename="$(find robotiq_description)/urdf/robotiq_2f_140_macro.urdf.xacro" />
-    <xacro:make_hand config_file_path="${config_file_path}"/>
+    <xacro:include filename="$(arg robotiq_description)/urdf/robotiq_2f_140_macro.urdf.xacro" />
+    <xacro:make_hand config_file="${config_file}"/>
 </robot>

File: robotiq_description/urdf/robotiq_2f_140_macro.urdf.xacro (robot description, xacro)
@@ -17,23 +17,4 @@
         gripper_max_force:=125.0
         gripper_closed_position:=0.695">
-        <!-- ros2 control include -->
-        <xacro:include filename="$(find robotiq_description)/urdf/2f_140.ros2_control.xacro" />
-        <!-- if we are simulating or directly communicating with the gripper we need a ros2 control instance -->
-        <xacro:if value="${include_ros2_control}">
-            <xacro:robotiq_gripper_ros2_control
-                name="${name}" prefix="${prefix}"
-                sim_gazebo="${sim_gazebo}"
-                sim_isaac="${sim_isaac}"
-                isaac_joint_commands="${isaac_joint_commands}"
-                isaac_joint_states="${isaac_joint_states}"
-                use_fake_hardware="${use_fake_hardware}"
-                mock_sensor_commands="${mock_sensor_commands}"
-                com_port="${com_port}"
-                gripper_speed_multiplier="${gripper_speed_multiplier}"
-                gripper_force_multiplier="${gripper_force_multiplier}"
-                gripper_max_speed="${gripper_max_speed}"
-                gripper_max_force="${gripper_max_force}"
-                gripper_closed_position="${gripper_closed_position}"/>
-        </xacro:if>
         <link name="${prefix}robotiq_140_base_link">
         <inertial>
@@ -65,9 +46,9 @@
     <xacro:right_outer_knuckle_joint prefix="${prefix}"/>
   </xacro:macro>
-  <xacro:macro name="make_hand" params="config_file_path">
-    <xacro:property name="cfg" value="${xacro.load_yaml(config_file_path)}"/>
+  <xacro:macro name="make_hand" params="config_file">
+    <xacro:property name="cfg" value="${xacro.load_yaml(config_file)}"/>
     <xacro:robotiq_gripper
         name="${cfg['info']['name'] if cfg['info']['name'] else 'Robotiq2F140'}"
-        prefix="${cfg['prefix']}"
+        prefix="${cfg['info']['prefix']}"
         sim_gazebo="${cfg['args']['sim_gazebo']}"
         sim_isaac="${cfg['args']['sim_isaac']}"

File: robotiq_description/urdf/robotiq_2f_85_config.urdf.xacro (robot description, xacro)
@@ -1,20 +1,19 @@
 <?xml version="1.0"?>
-<!-- Standalone URDF xacro that instantiates crab_claw_v1 -->
-<robot xmlns:xacro="http://www.ros.org/wiki/xacro" name="crab_claw_v1">
-    <xacro:include filename="$(find bam_descriptions)/urdf/common.xacro" />
-    <xacro:arg name="config_file_path" default="$(find bam_descriptions)/urdf/crab_claw_v1/config/crab_claw_skuBam_v0.0.0_config.yaml"/>
-    <xacro:property name="config_file_path" value="$(arg config_file_path)"/>
-    <xacro:property name="cfg" value="${xacro.load_yaml(config_file_path)}"/>
-    <xacro:property name="plugin" value="${cfg['plugin']}" />
-    <xacro:property name="reflect" value="${cfg['reflect']}" />
-    <xacro:property name="prefix" value="${cfg['prefix']}" />
-    <xacro:property name="world_xyz" value="${cfg['world_xyz']}" />
-    <xacro:property name="world_rpy" value="${cfg['world_rpy']}" />
-    <xacro:property name="base_xyz" value="${cfg['base_xyz']}" />
-    <xacro:property name="base_rpy" value="${cfg['base_rpy']}" />
-    <xacro:if value="${plugin != 'none'}">
+<robot xmlns:xacro="http://www.ros.org/wiki/xacro" name="robotiq_2f_85">
+    <xacro:arg name="robotiq_description" default="$(env ROBOTIQ_DESCRIPTION_PATH)" />
+    <xacro:arg name="config_file" default="$(arg robotiq_description)/urdf/config/robotiq_2f_85_2f_85_v0.0.0.yaml"/>
+    <xacro:property name="config_file" value="$(arg config_file)"/>
+    <xacro:property name="cfg" value="${xacro.load_yaml(config_file)}"/>
+    <xacro:property name="plugin" value="${cfg['args']['plugin']}" />
+    <xacro:property name="reflect" value="${cfg['args']['reflect']}" />
+    <xacro:property name="prefix" value="${cfg['info']['prefix']}" />
+    <xacro:property name="world_xyz" value="${cfg['args']['world_xyz']}" />
+    <xacro:property name="world_rpy" value="${cfg['args']['world_rpy']}" />
+    <xacro:property name="base_xyz" value="${cfg['args']['base_xyz']}" />
+    <xacro:property name="base_rpy" value="${cfg['args']['base_rpy']}" />
+    <!-- <xacro:if value="${plugin != 'none'}">
         <xacro:include filename="$(find bam_descriptions)/urdf/hybrid_v1/crab_claw_v1.ros2_control.xacro"/>
         <xacro:gripper_v1_ros2_control prefix="${prefix}" plugin="${plugin}"/>
-    </xacro:if>
+    </xacro:if> -->
     <link name="world"/>
     <joint name="world_to_base" type="fixed">
@@ -29,5 +28,5 @@
         <child link="${prefix}robotiq_85_base_link"/>
     </joint>
-    <xacro:include filename="$(find robotiq_description)/urdf/robotiq_2f_85_macro.urdf.xacro" />
-    <xacro:make_hand config_file_path="${config_file_path}"/>
+    <xacro:include filename="$(arg robotiq_description)/urdf/robotiq_2f_85_macro.urdf.xacro" />
+    <xacro:make_hand config_file="${config_file}"/>
 </robot>

File: robotiq_description/urdf/robotiq_2f_85_gripper.urdf.xacro (robot description, xacro)
@@ -5,5 +5,7 @@
     <xacro:arg name="com_port" default="/dev/ttyUSB0" />
     <!-- Import macros -->
-    <xacro:include filename="$(find robotiq_description)/urdf/robotiq_2f_85_macro.urdf.xacro" />
+    <!-- <xacro:arg name="robotiq_description" default="$(env ROBOTIQ_DESCRIPTION_PATH)" /> -->
+    <xacro:arg name="robotiq_description" default="$(find robotiq_description)" />
+    <xacro:include filename="$(arg robotiq_description)/urdf/robotiq_2f_85_macro.urdf.xacro" />
     <link name="world" />
     <xacro:robotiq_gripper

File: robotiq_description/urdf/robotiq_2f_85_macro.urdf.xacro (robot description, xacro)
@@ -1,4 +1,24 @@
 <?xml version="1.0"?>
 <robot xmlns:xacro="http://wiki.ros.org/xacro" name="robotiq_gripper">
+    <xacro:macro name="make_hand" params="config_file">
+        <xacro:property name="cfg" value="${xacro.load_yaml(config_file)}"/>
+        <xacro:robotiq_gripper
+            name="${cfg['info']['name'] if cfg['info']['name'] else 'RobotiqGripperHardwareInterface'}"
+            prefix="${cfg['info']['prefix']}"
+            sim_gazebo="${cfg['args']['sim_gazebo']}"
+            sim_isaac="${cfg['args']['sim_isaac']}"
+            isaac_joint_commands="${cfg['args']['isaac_joint_commands']}"
+            isaac_joint_states="${cfg['args']['isaac_joint_states']}"
+            use_fake_hardware="${cfg['args']['use_fake_hardware']}"
+            mock_sensor_commands="${cfg['args']['mock_sensor_commands']}"
+            include_ros2_control="${cfg['args']['include_ros2_control']}"
+            com_port="${cfg['args']['com_port']}"
+            gripper_speed_multiplier="${cfg['args']['gripper_speed_multiplier']}"
+            gripper_force_multiplier="${cfg['args']['gripper_force_multiplier']}"
+            gripper_max_speed="${cfg['args']['gripper_max_speed']}"
+            gripper_max_force="${cfg['args']['gripper_max_force']}"
+            gripper_closed_position="${cfg['args']['gripper_closed_position']}">
+        </xacro:robotiq_gripper>
+      </xacro:macro>
     <xacro:macro name="robotiq_gripper" params="
         name
@@ -17,23 +37,4 @@
         gripper_max_force:=235.0
         gripper_closed_position:=0.7929">
-        <!-- ros2 control include -->
-        <xacro:include filename="$(find robotiq_description)/urdf/2f_85.ros2_control.xacro" />
-        <!-- if we are simulating or directly communicating with the gripper we need a ros2 control instance -->
-        <xacro:if value="${include_ros2_control}">
-            <xacro:robotiq_gripper_ros2_control
-                name="${name}" prefix="${prefix}"
-                sim_gazebo="${sim_gazebo}"
-                sim_isaac="${sim_isaac}"
-                isaac_joint_commands="${isaac_joint_commands}"
-                isaac_joint_states="${isaac_joint_states}"
-                use_fake_hardware="${use_fake_hardware}"
-                mock_sensor_commands="${mock_sensor_commands}"
-                com_port="${com_port}"
-                gripper_speed_multiplier="${gripper_speed_multiplier}"
-                gripper_force_multiplier="${gripper_force_multiplier}"
-                gripper_max_speed="${gripper_max_speed}"
-                gripper_max_force="${gripper_max_force}"
-                gripper_closed_position="${gripper_closed_position}"/>
-        </xacro:if>
         <link name="${prefix}robotiq_85_base_link">
             <visual>
@@ -225,5 +226,7 @@
             </inertial>
         </link>
-        <joint name="${prefix}robotiq_85_left_knuckle_joint" type="revolute">
+        <!-- BUG ZILLA! https://github.com/stack-of-tasks/pinocchio/issues/2753 Alphabetical order screws it up.. -->
+        <!-- Previously called, but switch for something higher in alphabetical order: ${prefix}robotiq_85_left_knuckle_joint -->
+        <joint name="${prefix}finger_joint" type="revolute">
             <parent link="${prefix}robotiq_85_base_link" />
             <child link="${prefix}robotiq_85_left_knuckle_link" />
@@ -238,5 +241,5 @@
             <origin xyz="-0.03060114 0.0 0.05490452" rpy="0 0 0" />
             <limit lower="-0.8" upper="0.0" velocity="0.5" effort="50" />
-            <mimic joint="${prefix}robotiq_85_left_knuckle_joint" multiplier="-1" />
+            <mimic joint="${prefix}finger_joint" multiplier="-1" offset="0"/>
         </joint>
         <joint name="${prefix}robotiq_85_left_finger_joint" type="fixed">
@@ -250,52 +253,36 @@
             <origin xyz="-0.03152616 0.0 -0.00376347" rpy="0 0 0" />
         </joint>
-        <joint name="${prefix}robotiq_85_left_inner_knuckle_joint" type="continuous">
+        <joint name="${prefix}robotiq_85_left_inner_knuckle_joint" type="revolute">
             <parent link="${prefix}robotiq_85_base_link" />
             <child link="${prefix}robotiq_85_left_inner_knuckle_link" />
             <axis xyz="0 -1 0" />
             <origin xyz="0.0127 0.0 0.06142" rpy="0 0 0" />
-            <mimic joint="${prefix}robotiq_85_left_knuckle_joint" />
-        </joint>
-        <joint name="${prefix}robotiq_85_right_inner_knuckle_joint" type="continuous">
+            <mimic joint="${prefix}finger_joint" multiplier="1" offset="0"/>
+            <limit lower="${-2*pi}" upper="${2*pi}" velocity="0.5" effort="50" />
+        </joint>
+        <joint name="${prefix}robotiq_85_right_inner_knuckle_joint" type="revolute">
             <parent link="${prefix}robotiq_85_base_link" />
             <child link="${prefix}robotiq_85_right_inner_knuckle_link" />
             <axis xyz="0 -1 0" />
             <origin xyz="-0.0127 0.0 0.06142" rpy="0 0 0" />
-            <mimic joint="${prefix}robotiq_85_left_knuckle_joint" multiplier="-1" />
-        </joint>
-        <joint name="${prefix}robotiq_85_left_finger_tip_joint" type="continuous">
+            <mimic joint="${prefix}finger_joint" multiplier="-1" offset="0"/>
+            <limit lower="${-2*pi}" upper="${2*pi}" velocity="0.5" effort="50" />
+        </joint>
+        <joint name="${prefix}robotiq_85_left_finger_tip_joint" type="revolute">
             <parent link="${prefix}robotiq_85_left_finger_link" />
             <child link="${prefix}robotiq_85_left_finger_tip_link" />
             <axis xyz="0 -1 0" />
             <origin xyz="0.00563134 0.0 0.04718515" rpy="0 0 0" />
-            <mimic joint="${prefix}robotiq_85_left_knuckle_joint" multiplier="-1" />
-        </joint>
-        <joint name="${prefix}robotiq_85_right_finger_tip_joint" type="continuous">
+            <mimic joint="${prefix}finger_joint" multiplier="-1" offset="0"/>
+            <limit lower="${-2*pi}" upper="${2*pi}" velocity="0.5" effort="50" />
+        </joint>
+        <joint name="${prefix}robotiq_85_right_finger_tip_joint" type="revolute">
             <parent link="${prefix}robotiq_85_right_finger_link" />
             <child link="${prefix}robotiq_85_right_finger_tip_link" />
             <axis xyz="0 -1 0" />
             <origin xyz="-0.00563134 0.0 0.04718515" rpy="0 0 0" />
-            <mimic joint="${prefix}robotiq_85_left_knuckle_joint" />
+            <mimic joint="${prefix}finger_joint" multiplier="1" offset="0"/>
+            <limit lower="${-2*pi}" upper="${2*pi}" velocity="0.5" effort="50" />
     </joint>
   </xacro:macro>
-  <xacro:macro name="make_hand" params="config_file_path">
-    <xacro:property name="cfg" value="${xacro.load_yaml(config_file_path)}"/>
-    <xacro:robotiq_gripper
-        name="${cfg['info']['name'] if cfg['info']['name'] else 'RobotiqGripperHardwareInterface'}"
-        prefix="${cfg['prefix']}"
-        sim_gazebo="${cfg['args']['sim_gazebo']}"
-        sim_isaac="${cfg['args']['sim_isaac']}"
-        isaac_joint_commands="${cfg['args']['isaac_joint_commands']}"
-        isaac_joint_states="${cfg['args']['isaac_joint_states']}"
-        use_fake_hardware="${cfg['args']['use_fake_hardware']}"
-        mock_sensor_commands="${cfg['args']['mock_sensor_commands']}"
-        include_ros2_control="${cfg['args']['include_ros2_control']}"
-        com_port="${cfg['args']['com_port']}"
-        gripper_speed_multiplier="${cfg['args']['gripper_speed_multiplier']}"
-        gripper_force_multiplier="${cfg['args']['gripper_force_multiplier']}"
-        gripper_max_speed="${cfg['args']['gripper_max_speed']}"
-        gripper_max_force="${cfg['args']['gripper_max_force']}"
-        gripper_closed_position="${cfg['args']['gripper_closed_position']}">
-    </xacro:robotiq_gripper>
-  </xacro:macro>
 </robot>
