Commit message: ss

File: robotiq_description/urdf/robotiq_2f_140_macro.urdf.xacro (robot description, xacro)
@@ -46,4 +46,7 @@
     <xacro:right_outer_knuckle_joint prefix="${prefix}"/>
   </xacro:macro>
+  <xacro:macro name="make_config" params="config_file">
+    <xacro:make_hand config_file="${config_file}"/>
+  </xacro:macro>
   <xacro:macro name="make_hand" params="config_file">
     <xacro:property name="cfg" value="${xacro.load_yaml(config_file)}"/>

File: robotiq_description/urdf/robotiq_2f_85_macro.urdf.xacro (robot description, xacro)
@@ -1,4 +1,7 @@
 <?xml version="1.0"?>
 <robot xmlns:xacro="http://wiki.ros.org/xacro" name="robotiq_gripper">
+    <xacro:macro name="make_config" params="config_file">
+        <xacro:make_hand config_file="${config_file}"/>
+    </xacro:macro>
     <xacro:macro name="make_hand" params="config_file">
         <xacro:property name="cfg" value="${xacro.load_yaml(config_file)}"/>
